Commit message: kabot hostile takeover

File: src/kabot_description/models/diff_drive/gazebo_control.xacro (robot description, xacro)
@@ -3,19 +3,23 @@
     <!-- DIFF DRIVE SIMULATION -->
     <gazebo>
-        <plugin name="diff_drive" filename="libgazebo_ros_diff_drive.so">
-            <left_joint>left_wheel_joint</left_joint>
-            <right_joint>right_wheel_joint</right_joint>
-            <wheel_separation>0.13</wheel_separation>
-            <wheel_diameter>0.07</wheel_diameter>
-            <max_wheel_torque>1</max_wheel_torque>
-            <max_wheel_acceleration>0.5</max_wheel_acceleration>
-            <odometry_frame>odom</odometry_frame>
-            <robot_base_frame>base_link</robot_base_frame>
-            <publish_odom>true</publish_odom>
-            <publish_odom_tf>true</publish_odom_tf>
-            <publish_wheel_tf>true</publish_wheel_tf>
-        </plugin>
+      <plugin
+        filename="ignition-gazebo-diff-drive-system"
+        name="ignition::gazebo::systems::DiffDrive">
+        <left_joint>left_wheel_joint</left_joint>
+        <right_joint>right_wheel_joint</right_joint>
+        <wheel_separation>0.13</wheel_separation>
+        <wheel_radius>0.35</wheel_radius>
+        <odom_publish_frequency>1</odom_publish_frequency>
+        <max_linear_acceleration>1</max_linear_acceleration>
+        <min_linear_acceleration>-1</min_linear_acceleration>
+        <max_angular_acceleration>2</max_angular_acceleration>
+        <min_angular_acceleration>-2</min_angular_acceleration>
+        <max_linear_velocity>0.5</max_linear_velocity>
+        <min_linear_velocity>-0.5</min_linear_velocity>
+        <max_angular_velocity>1</max_angular_velocity>
+        <min_angular_velocity>-1</min_angular_velocity>
+      </plugin>
     </gazebo>
-    <!-- ARUCO SIMULATION-->
+    <!-- ARUCO SIMULATION
     <link name="aruco_link">
         <visual>
@@ -40,4 +44,4 @@
         <child link="aruco_link"/>
         <origin xyz="0 0 0.036" rpy="0 ${pi} 0"/>
-    </joint>
+    </joint> -->
 </robot>
