Commit message: spawn_kabot

File: src/kabot_description/urdf/gazebo_control.xacro (robot description, xacro)
@@ -1,47 +1,22 @@
 <?xml version="1.0"?>
 <robot xmlns:xacro="http://www.ros.org/wiki/xacro">
-    <!-- DIFF DRIVE SIMULATION -->
     <gazebo>
-      <plugin
-        filename="ignition-gazebo-diff-drive-system"
-        name="ignition::gazebo::systems::DiffDrive">
-        <left_joint>left_wheel_joint</left_joint>
-        <right_joint>right_wheel_joint</right_joint>
-        <wheel_separation>0.13</wheel_separation>
-        <wheel_radius>0.35</wheel_radius>
-        <odom_publish_frequency>1</odom_publish_frequency>
-        <max_linear_acceleration>1</max_linear_acceleration>
-        <min_linear_acceleration>-1</min_linear_acceleration>
-        <max_angular_acceleration>2</max_angular_acceleration>
-        <min_angular_acceleration>-2</min_angular_acceleration>
-        <max_linear_velocity>0.5</max_linear_velocity>
-        <min_linear_velocity>-0.5</min_linear_velocity>
-        <max_angular_velocity>1</max_angular_velocity>
-        <min_angular_velocity>-1</min_angular_velocity>
-      </plugin>
+        <plugin name="joint_controller" filename="libgazebo_ros_joint_controller.so">
+            <ros>
+            <namespace>/kabot</namespace>
+            <remapping>
+                <remap from="joint_states" to="/kabot/wheels" />
+            </remapping>
+            </ros>
+            <update_rate>100</update_rate>
+            <joint>
+            <name>left_wheel_joint</name>
+            <type>velocity</type>
+            </joint>
+            <joint>
+            <name>right_wheel_joint</name>
+            <type>velocity</type>
+            </joint>
+        </plugin>
     </gazebo>
-    <!-- ARUCO SIMULATION
-    <link name="aruco_link">
-        <visual>
-            <geometry>
-                <mesh filename="file://$(find kabot_launcher)/description/meshes/aruco.dae" scale="0.03 0.03 0.03"/>
-            </geometry>
-        </visual>
-        <collision>
-            <geometry>
-                <box size="0.05 0.05 0.01"/>
-            </geometry>
-        </collision>
-        <xacro:inertial_box mass="0.0001" x="0.0001" y="0.0001" z="0.0001">
-            <origin xyz="0 0 0" rpy="0 0 0"/>
-        </xacro:inertial_box>
-    </link>
-    <gazebo reference="aruco_link">
-        <material>aruco</material>
-    </gazebo>
-    <joint name="aruco_link" type="fixed">
-        <parent link="chassis_link"/>
-        <child link="aruco_link"/>
-        <origin xyz="0 0 0.036" rpy="0 ${pi} 0"/>
-    </joint> -->
 </robot>

File: src/kabot_description/urdf/kabot.xacro (robot description, xacro)
@@ -5,4 +5,4 @@
     <xacro:wheel name="left_wheel" origin="0 ${chassis_radius+0.005} -0.005" parent="chassis_link" direction="1"/>
     <xacro:wheel name="right_wheel" origin="0 -${chassis_radius+0.005} -0.005" parent="chassis_link" direction="1"/>
-    <!-- <xacro:include filename="gazebo_control.xacro"/> -->
+    <xacro:include filename="gazebo_control.xacro"/>
 </robot>
